File: hardware/rotary_encoder.kicad_pcb (KiCad board)
At the start: 2 copper layers, 30 x 25 mm, 20 parts, among them P1 CON-SENSOR2, P2 BOOT, P3 DEBUG, U1 XMC1XXX24, U2 ROTARY_ENCODER, U3 DRILL, U4 DRILL, U5 DRILL, U6 DRILL

Commit message: Add logos
Parts:
- added G***: LOGO, kicad-libraries:Logo_CoMCU, B.Cu at (67.8, 42.3)
- added VAL: WEEE_7mm, kicad-libraries:WEEE_7mm, B.Cu at (48.4, 42.3)
- added VAL: CE_5mm, kicad-libraries:CE_5mm, B.Cu at (61.5, 42.3)

Commit message: change led position
Parts:
- moved R1 2.26 mm to (57.9, 52.0)
- moved D1 2.25 mm to (61.0, 52.0)
Routing:
- net Net-(R1-Pad1): track 2.81 -> 4.89 mm
Changed lines of the file:
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@@
-(kicad_pcb (version 4) (host pcbnew 4.0.2+dfsg1-stable)
+(kicad_pcb (version 4) (host pcbnew 4.0.7-e2-6376~58~ubuntu17.04.1)
   (general
     (links 45)
-    (no_connects 1)
-    (area 42.709499 29.609499 73.090501 54.990501)
+    (no_connects 0)
+    (area 42.044999 28.944999 282.27147 165.489573)
     (thickness 1.6002)
     (drawings 12)
-    (tracks 147)
+    (tracks 148)
     (zones 0)
     (modules 23)
@@
   (layers
     (0 Vorderseite jumper)
-    (31 Rückseite jumper)
+    (31 Rückseite jumper hide)
     (32 B.Adhes user)
     (33 F.Adhes user)
@@
   )
   (setup
-    (last_trace_width 0.29972)
+    (last_trace_width 0.25)
     (user_trace_width 0.2)
     (user_trace_width 0.25)
@@
   )
   (module kicad-libraries:D0603E (layer Vorderseite)
-    (at 61.1 49.8 180)
+    (at 61 52.05 180)
     (attr smd)
     (fp_text reference D1 (at 0.85 0.45 180) (layer F.Fab)
@@
   )
   (module kicad-libraries:R0603F (layer Vorderseite)
-    (at 58.1 49.8)
+    (at 57.9 52.05)
     (attr smd)
     (fp_text reference R1 (at 0.05 0.225) (layer F.Fab)
@@
       (xy 1.301301 2.715081) (xy 1.302426 2.714986)) (layer B.SilkS) (width 0.01))
   )
-  (gr_text status (at 61.15 51.05) (layer F.SilkS)
+  (gr_text status (at 61 50.75) (layer F.SilkS)
     (effects (font (size 0.7 0.7) (thickness 0.12)))
   )
@@
     (effects (font (size 0.8 0.8) (thickness 0.15)))
   )
-  (gr_text "Rotary Encoder 2.0\n" (at 57.9 53) (layer F.SilkS)
+  (gr_text "Rotary Encoder 2.0\n" (at 57.9 53.55) (layer F.SilkS)
     (effects (font (size 0.8 0.8) (thickness 0.15)))
   )
@@
   (via (at 44.1 47.2) (size 0.55) (drill 0.25) (layers Vorderseite Rückseite) (net 1))
   (segment (start 56.65 42.3) (end 57.25 42.3) (width 0.29972) (layer Rückseite) (net 1))
+  (segment (start 61.8501 52.05) (end 61.8501 52.7999) (width 0.25) (layer Vorderseite) (net 2))
+  (segment (start 54.65 52.5) (end 54 52.5) (width 0.25) (layer Vorderseite) (net 2))
+  (segment (start 55.6 53.45) (end 54.65 52.5) (width 0.25) (layer Vorderseite) (net 2))
+  (segment (start 61.2 53.45) (end 55.6 53.45) (width 0.25) (layer Vorderseite) (net 2))
+  (segment (start 61.8501 52.7999) (end 61.2 53.45) (width 0.25) (layer Vorderseite) (net 2))
   (segment (start 47.7 49.6) (end 50.6 52.5) (width 0.25) (layer Vorderseite) (net 2))
   (segment (start 51.4 41.5) (end 51.2 41.7) (width 0.25) (layer Vorderseite) (net 2))
@@
   (segment (start 52.9491 41.20122) (end 52.9491 41.99878) (width 0.25) (layer Vorderseite) (net 2))
   (segment (start 52.9491 41.99878) (end 52.9491 42.79888) (width 0.25) (layer Vorderseite) (net 2))
-  (segment (start 54.25 51.7) (end 55.7 51.7) (width 0.25) (layer Vorderseite) (net 2))
-  (segment (start 55.7 51.7) (end 56.5 50.9) (width 0.25) (layer Vorderseite) (net 2))
-  (segment (start 56.5 50.9) (end 61.5 50.9) (width 0.25) (layer Vorderseite) (net 2))
-  (segment (start 61.5 50.9) (end 61.9501 50.4499) (width 0.25) (layer Vorderseite) (net 2))
-  (segment (start 61.9501 50.4499) (end 61.9501 49.8) (width 0.25) (layer Vorderseite) (net 2))
   (segment (start 49.8 40.75) (end 51.3 40.75) (width 0.5) (layer Vorderseite) (net 2))
   (segment (start 51.3 40.75) (end 51.4 40.65) (width 0.5) (layer Vorderseite) (net 2))
@@
   (segment (start 53.75 50.85) (end 54.25 51.35) (width 0.25) (layer Vorderseite) (net 2))
   (segment (start 54.25 51.35) (end 54.25 51.7) (width 0.25) (layer Vorderseite) (net 2))
-  (segment (start 58.85 49.8) (end 60.2499 49.8) (width 0.25) (layer Vorderseite) (net 3))
+  (segment (start 58.65 52.05) (end 60.1499 52.05) (width 0.25) (layer Vorderseite) (net 3))
   (segment (start 47.5 42.3) (end 48.5 42.3) (width 0.25) (layer Vorderseite) (net 5))
   (segment (start 49.2507 43.5507) (end 49.925 43.5507) (width 0.25) (layer Vorderseite) (net 5))
@@
   (segment (start 48.95108 44.54892) (end 49.925 44.54892) (width 0.25) (layer Vorderseite) (net 7))
   (segment (start 48.7 44.8) (end 48.95108 44.54892) (width 0.25) (layer Vorderseite) (net 7))
+  (segment (start 49.25 49) (end 49.65 49) (width 0.25) (layer Vorderseite) (net 8))
   (segment (start 51.475 48.85) (end 50.55 48.85) (width 0.25) (layer Vorderseite) (net 8))
   (segment (start 50.4 49) (end 49.25 49) (width 0.25) (layer Vorderseite) (net 8))
@@
   (segment (start 50.4 49.75) (end 50.4 50.55) (width 0.25) (layer Vorderseite) (net 9))
   (segment (start 50.8 49.35) (end 50.4 49.75) (width 0.25) (layer Vorderseite) (net 9))
-  (segment (start 55.525 48.35) (end 56.55 48.35) (width 0.25) (layer Vorderseite) (net 10))
-  (segment (start 57.35 49.15) (end 57.35 49.8) (width 0.25) (layer Vorderseite) (net 10))
-  (segment (start 56.55 48.35) (end 57.35 49.15) (width 0.25) (layer Vorderseite) (net 10))
+  (segment (start 55.525 48.35) (end 56.4 48.35) (width 0.25) (layer Vorderseite) (net 10))
+  (segment (start 57.15 49.1) (end 57.15 52.05) (width 0.25) (layer Vorderseite) (net 10))
+  (segment (start 56.4 48.35) (end 57.15 49.1) (width 0.25) (layer Vorderseite) (net 10))
   (segment (start 51.075 45.0493) (end 51.511968 45.0493) (width 0.25) (layer Vorderseite) (net 11))
   (segment (start 51.475 46.225) (end 51.475 46.85) (width 0.25) (layer Vorderseite) (net 11))
@@
     (polygon
       (pts
-        (xy 72.8 54.8) (xy 42.9 54.8) (xy 42.9 29.8) (xy 72.9 29.8) (xy 72.8 54.8)
+        (xy 72.8 54.8) (xy 42.9 54.8) (xy 42.9 29.8) (xy 72.9 29.8)
       )
     )

Commit message: fix debug pin connection
Parts:
- moved P3 7.38 mm to (53.8, 44.0)
Connections:
- P1 pad 1: Net-(P1-Pad1) -> (no net)
- RP2 pad 2: Net-(RP2-Pad2) -> (no net)
- U1 pad 11: Net-(U1-Pad11) -> (no net)
- U1 pad 12: Net-(U1-Pad12) -> (no net)
- U1 pad 13: Net-(U1-Pad13) -> (no net)
- U1 pad 14: Net-(U1-Pad14) -> (no net)
- U1 pad 16: Net-(U1-Pad16) -> (no net)
- U1 pad 17: Net-(U1-Pad17) -> (no net)
- U1 pad 18: Net-(U1-Pad18) -> (no net)
- U1 pad 19: Net-(U1-Pad19) -> Net-(P3-Pad1)
- U1 pad 20: Net-(U1-Pad20) -> (no net)
- U1 pad 21: Net-(U1-Pad21) -> (no net)
- U1 pad 4: Net-(U1-Pad4) -> (no net)
- U1 pad 6: Net-(P3-Pad1) -> (no net)
- U1 pad 8: Net-(U1-Pad8) -> (no net)

Commit message: add rc capacitors, mode debug
 * add two 10nF capacitors to a,b to remove glitches
 * move debug pin
Parts:
- added C5: 10nF, kicad-libraries:C0603F, F.Cu at (55.1, 43.1)
- added C6: 10nF, kicad-libraries:C0603F, F.Cu at (55.1, 40.1)
- moved P3 5.26 mm to (57.1, 48.0)
- moved C2 4.14 mm to (50.5, 35.9), turned to 180 degrees
- moved C1 2.42 mm to (50.5, 37.5), turned to 180 degrees
- moved RP2 1.54 mm to (52.4, 41.0)
Connections:
- U1 pad 16: (no net) -> Net-(P3-Pad1)
- U1 pad 19: Net-(P3-Pad1) -> (no net)
Routing:
- net VCC: track 42.2 -> 51.4 mm
- net GND: track 20.4 -> 27.2 mm, vias 6 -> 7
- net SW1: track 29.6 -> 32.0 mm, vias 2 -> 3
- net IN_B: track 14.9 -> 16.7 mm
- net IN_A: track 16.2 -> 17.7 mm
- net Net-(P3-Pad1): track 2.47 -> 1.71 mm

Commit message: specify processor type
Parts:
- U1: value XMC1XXX24 -> XMC110024
Changed lines of the file:
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@@
       (effects (font (size 0.3 0.3) (thickness 0.075)))
     )
-    (fp_text value XMC1XXX24 (at 0 0.8) (layer F.Fab)
+    (fp_text value XMC110024 (at 0 0.8) (layer F.Fab)
       (effects (font (size 0.3 0.3) (thickness 0.075)))
     )
