File: hardware/rotary-encoder-v2.kicad_sch (KiCad schematic)
At the start: 19 parts

Commit message: fix symbol libraries
Parts:
- C1: value (none) -> 10uF; footprint (none) -> kicad-libraries:C0805E; symbol C -> tinkerforge:C
- C2: value (none) -> 1uF; footprint (none) -> kicad-libraries:C0603F; symbol C -> tinkerforge:C
- C3: value (none) -> 100nF; footprint (none) -> kicad-libraries:C0603F; symbol C -> tinkerforge:C
- C4: value (none) -> 220pF; footprint (none) -> kicad-libraries:C0402F; symbol C -> tinkerforge:C
- C5, C6: value (none) -> 10nF; footprint (none) -> kicad-libraries:C0603F; symbol C -> tinkerforge:C
- D1: value (none) -> blue; footprint (none) -> kicad-libraries:D0603F; symbol LED -> tinkerforge:LED
- P1: value (none) -> CON-SENSOR2; footprint (none) -> kicad-libraries:CON-SENSOR2; symbol CON-SENSOR2 -> tinkerforge:CON-SENSOR2
- P2: value (none) -> BOOT; footprint (none) -> kicad-libraries:SolderJumper; symbol CONN_01X02 -> tinkerforge:CONN_01X02
- P3: value (none) -> DEBUG; footprint (none) -> kicad-libraries:DEBUG_PAD; symbol CONN_01X01 -> tinkerforge:CONN_01X01
- R1: value (none) -> 1k; footprint (none) -> kicad-libraries:R0603F; symbol R -> tinkerforge:R
- RP1: value (none) -> 82; footprint (none) -> kicad-libraries:4X0402; symbol R_PACK4 -> tinkerforge:R_PACK4
- RP2: value (none) -> 10k; footprint (none) -> kicad-libraries:4X0603; symbol R_PACK4 -> tinkerforge:R_PACK4
- U1: value (none) -> XMC110024; footprint (none) -> kicad-libraries:QFN24-4x4mm-0.5mm; symbol XMC1XXX24 -> tinkerforge:XMC1XXX24
- U2: value (none) -> ROTARY_ENCODER; footprint (none) -> kicad-libraries:ROTARY_ENCODER; symbol ROTARY_ENCODER -> tinkerforge:ROTARY_ENCODER
- U3, U4, U5, U6: value (none) -> DRILL; footprint (none) -> kicad-libraries:DRILL_NP; symbol DRILL -> tinkerforge:DRILL
Connections:
- net IN_A: now also C6.1, RP2.1 (P1), U1.2 (P2.1_AIO), U2.A (IN_A)
- net IN_B: now also C5.1, RP2.3 (P3), U1.3 (P2.2_AI), U2.B (IN_B)
- net S-CLK: now also RP1.7 (R2), U1.23 (P0.14_IO)
- net S-CS: now also RP1.8 (R1), U1.22 (P0.13_IO)
- net S-MISO: now also RP1.5 (R4), U1.1 (P2.0_AIO)
- net S-MOSI: now also RP1.6 (R3), U1.24 (P0.15_IO)
- net SW1: now also RP2.4 (P4), U1.7 (P2.10_AIO), U2.SW1
- new net: P1.4, RP1.1 (P1)
- new net: P1.5, RP1.2 (P2)
- new net: P1.6, RP1.3 (P3)
- new net: C4.1, P1.7, RP1.4 (P4)
- new net: R1.1, U1.15 (P0.0_IO)
- new net: P3.1 (P1), U1.16 (P0.5_IO)
- new net: P2.2 (P2), U1.5 (P2.7/P2.8_AI)
- new net: D1.2 (K), R1.2
- new net GND: C1.2, C2.2, C3.2, C4.2, C5.2, C6.2, P1.2, P1.EP, P2.1 (P1), U1.9 (VSSP/VSS), U1.EXP (VSSP), U2.C (COM), U2.SW2
- new net VCC: C1.1, C2.1, C3.1, D1.1 (A), P1.3, RP2.5 (R4), RP2.8 (R1), U1.10 (VDDP/VDD)

Commit message: Data Cleanup
Other:
- note added: "Copyright Tinkerforge GmbH 2023. This documentation describes Open Hardware and is licensed under the CERN OHL v. 1.1. You may redistribute and modify this documentation under the terms of the CERN OHL v.1.1. (http://ohwr.org/cernohl). This documentation is distributed WITHOUT ANY EXPRESS OR IMPLIED WARRANTY, INCLUDING OF MERCHANTABILITY, SATISFACTORY QUALITY AND FITNESS FOR A PARTICULAR PURPOSE.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"
- note removed: "Copyright Tinkerforge GmbH 2017. This documentation describes Open Hardware and is licensed under the CERN OHL v. 1.1. You may redistribute and modify this documentation under the terms of the CERN OHL v.1.1. (http://ohwr.org/cernohl). This documentation is distributed WITHOUT ANY EXPRESS OR IMPLIED WARRANTY, INCLUDING OF MERCHANTABILITY, SATISFACTORY QUALITY AND FITNESS FOR A PARTICULAR PURPOSE.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"
Changed lines of the file:
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@@
   (title_block
     (title "Rotary Encoder Bricklet")
-    (date "2017-09-18")
+    (date "2023-01-26")
     (rev "2.0")
     (company "Tinkerforge GmbH")
     (comment 1 "Licensed under CERN OHL v.1.1")
-    (comment 2 "Copyright (©) 2017, L.Lauer <lukas@tinkerforge.com>")
+    (comment 2 "Copyright (©) 2023, T.Schneidermann <tim@tinkerforge.com>")
   )
   (junction (at 62.23 26.67) (diameter 0) (color 0 0 0 0)
@@
     (effects (font (size 0.9906 0.9906)) (justify left bottom))
   )
-  (text "Copyright Tinkerforge GmbH 2017.\nThis documentation describes Open Hardware and is licensed under the\nCERN OHL v. 1.1.\nYou may redistribute and modify this documentation under the terms of the\nCERN OHL v.1.1. (http://ohwr.org/cernohl). This documentation is distributed\nWITHOUT ANY EXPRESS OR IMPLIED WARRANTY, INCLUDING OF\nMERCHANTABILITY, SATISFACTORY QUALITY AND FITNESS FOR A\nPARTICULAR PURPOSE. Please see the CERN OHL v.1.1 for applicable\nconditions\n"
+  (text "Copyright Tinkerforge GmbH 2023.\nThis documentation describes Open Hardware and is licensed under the\nCERN OHL v. 1.1.\nYou may redistribute and modify this documentation under the terms of the\nCERN OHL v.1.1. (http://ohwr.org/cernohl). This documentation is distributed\nWITHOUT ANY EXPRESS OR IMPLIED WARRANTY, INCLUDING OF\nMERCHANTABILITY, SATISFACTORY QUALITY AND FITNESS FOR A\nPARTICULAR PURPOSE. Please see the CERN OHL v.1.1 for applicable\nconditions\n"
     (at 12.7 196.85 0)
     (effects (font (size 1.016 1.016)) (justify left bottom))
